File: Qwiic_Multi_Port_Board/Production/Qwiic_Multi_Port_Board-Panel.brd (EAGLE design)
At the start: 97.3 x 97.3 mm, 122 parts, among them J1 QWIIC_RIGHT_ANGLE, J10 QWIIC_RIGHT_ANGLE, J11 QWIIC_RIGHT_ANGLE, J12 QWIIC_RIGHT_ANGLE, J13 QWIIC_RIGHT_ANGLE, J14 QWIIC_RIGHT_ANGLE, J15 QWIIC_RIGHT_ANGLE, J16 QWIIC_RIGHT_ANGLE, J17 QWIIC_RIGHT_ANGLE, J18 QWIIC_RIGHT_ANGLE, J19 QWIIC_RIGHT_ANGLE, J2 QWIIC_RIGHT_ANGLE, J20 QWIIC_RIGHT_ANGLE, J21 QWIIC_RIGHT_ANGLE, J22 QWIIC_RIGHT_ANGLE, J23 QWIIC_RIGHT_ANGLE, J24 QWIIC_RIGHT_ANGLE, J25 QWIIC_RIGHT_ANGLE, J26 QWIIC_RIGHT_ANGLE, J27 QWIIC_RIGHT_ANGLE, J28 QWIIC_RIGHT_ANGLE, J29 QWIIC_RIGHT_ANGLE, J3 QWIIC_RIGHT_ANGLE, J30 QWIIC_RIGHT_ANGLE, J31 QWIIC_RIGHT_ANGLE, J32 QWIIC_RIGHT_ANGLE, J33 QWIIC_RIGHT_ANGLE, J34 QWIIC_RIGHT_ANGLE, J35 QWIIC_RIGHT_ANGLE, J36 QWIIC_RIGHT_ANGLE, J4 QWIIC_RIGHT_ANGLE, J5 QWIIC_RIGHT_ANGLE, J6 QWIIC_RIGHT_ANGLE, J7 QWIIC_RIGHT_ANGLE, J8 QWIIC_RIGHT_ANGLE, J9 QWIIC_RIGHT_ANGLE

Commit message: Created panel and generated gerbers
Parts:
- removed E$1, E$2, E$3, E$4: (no value), SparkFun-Aesthetics:FIDUCIAL-1X2
- removed E$5: (no value), SparkFun-Retired:FIDUCIAL-1.5X3
- added H19, H20, H21, H22, H23, H24, H25, H26, H27, H28, H29, H30, H31, H32, H33, H34, H35, H36, H37, H38, H39, H40, H41, H42, H43, H44, H45, H46, H47, H48, H49, H50: STAND-OFFTIGHT, SparkFun-Hardware:STAND-OFF-TIGHT
- added J100, J37, J38, J39, J40, J41, J42, J43, J44, J45, J46, J47, J48, J49, J50, J51, J52, J53, J54, J55, J56, J57, J58, J59, J60, J61, J62, J63, J64, J65, J66, J67, J68, J69, J70, J71, J72, J73, J74, J75, J76, J77, J78, J79, J80, J81, J82, J83, J84, J85, J86, J87, J88, J89, J90, J91, J92, J93, J94, J95, J96, J97, J98, J99: QWIIC_RIGHT_ANGLE, SparkFun-Connectors:JST04_1MM_RA
- added U$100, U$104, U$107, U$111, U$114, U$118, U$121, U$125, U$128, U$132, U$135, U$139, U$142, U$146, U$149, U$153, U$156, U$160, U$163, U$167, U$170, U$174, U$65, U$69, U$72, U$76, U$79, U$83, U$86, U$90, U$93, U$97: (no value), buzzard_labels (75):MULTI1
- added U$101, U$105, U$108, U$112, U$115, U$119, U$122, U$126, U$129, U$133, U$136, U$140, U$143, U$147, U$150, U$154, U$157, U$161, U$164, U$168, U$171, U$175, U$66, U$70, U$73, U$77, U$80, U$84, U$87, U$91, U$94, U$98: (no value), buzzard_labels (75):PORT2
- added U$102, U$103, U$109, U$110, U$116, U$117, U$123, U$124, U$130, U$131, U$137, U$138, U$144, U$145, U$151, U$152, U$158, U$159, U$165, U$166, U$172, U$173, U$67, U$68, U$74, U$75, U$81, U$82, U$88, U$89, U$95, U$96: (no value), SparkFun-Aesthetics:QWIIC_6MM
- added U$106, U$113, U$120, U$127, U$134, U$141, U$148, U$155, U$162, U$169, U$64, U$71, U$78, U$85, U$92, U$99: (no value), SparkX:SPARKX-SMALL
- moved H10 81.9 mm to (112.5, 8.89)
- moved H8 81.9 mm to (86.6, 8.89)
- moved J13 81.9 mm to (90.4, 5.08)
- moved J14 81.9 mm to (82.8, 12.7)
- moved J16 81.9 mm to (90.4, 20.3)
- moved J18 81.9 mm to (108.7, 12.7)
- moved U$22 81.9 mm to (90.4, 5.59)
- moved U$23 81.9 mm to (85.9, 11.8)
- moved U$24 81.9 mm to (90.2, 11.8)
- moved U$25 81.9 mm to (90.4, 13.8)
- moved U$26 81.9 mm to (90.4, 13.8)
- moved U$27 81.9 mm to (95.1, 11.8)
- moved U$30 81.9 mm to (111.8, 11.8)
- moved U$31 81.9 mm to (116.1, 11.8)
- moved U$34 81.9 mm to (121.0, 11.8)
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Connections:
- new net 3.3V10: J41.2, J42.2, J43.2, J44.2
- new net 3.3V11: J45.2, J46.2, J47.2, J48.2
- new net 3.3V12: J49.2, J50.2, J51.2, J52.2
- new net 3.3V13: J53.2, J54.2, J55.2, J56.2
- new net 3.3V14: J57.2, J58.2, J59.2, J60.2
- new net 3.3V15: J61.2, J62.2, J63.2, J64.2
- new net 3.3V16: J65.2, J66.2, J67.2, J68.2
- new net 3.3V17: J69.2, J70.2, J71.2, J72.2
- new net 3.3V18: J73.2, J74.2, J75.2, J76.2
- new net 3.3V19: J77.2, J78.2, J79.2, J80.2
- new net 3.3V20: J81.2, J82.2, J83.2, J84.2
- new net 3.3V21: J85.2, J86.2, J87.2, J88.2
- new net 3.3V22: J89.2, J90.2, J91.2, J92.2
- new net 3.3V23: J93.2, J94.2, J95.2, J96.2
- new net 3.3V24: J100.2, J97.2, J98.2, J99.2
- new net 3.3V9: J37.2, J38.2, J39.2, J40.2
- new net GND10: J41.1, J42.1, J43.1, J44.1
- new net GND11: J45.1, J46.1, J47.1, J48.1
- new net GND12: J49.1, J50.1, J51.1, J52.1
- new net GND13: J53.1, J54.1, J55.1, J56.1
- new net GND14: J57.1, J58.1, J59.1, J60.1
- new net GND15: J61.1, J62.1, J63.1, J64.1
- new net GND16: J65.1, J66.1, J67.1, J68.1
- new net GND17: J69.1, J70.1, J71.1, J72.1
- new net GND18: J73.1, J74.1, J75.1, J76.1
- new net GND19: J77.1, J78.1, J79.1, J80.1
- new net GND20: J81.1, J82.1, J83.1, J84.1
- new net GND21: J85.1, J86.1, J87.1, J88.1
- new net GND22: J89.1, J90.1, J91.1, J92.1
- new net GND23: J93.1, J94.1, J95.1, J96.1
- new net GND24: J100.1, J97.1, J98.1, J99.1
- new net GND9: J37.1, J38.1, J39.1, J40.1
- new net SCL10: J41.4, J42.4, J43.4, J44.4
- new net SCL11: J45.4, J46.4, J47.4, J48.4
- new net SCL12: J49.4, J50.4, J51.4, J52.4
- new net SCL13: J53.4, J54.4, J55.4, J56.4
- new net SCL14: J57.4, J58.4, J59.4, J60.4
- new net SCL15: J61.4, J62.4, J63.4, J64.4
- new net SCL16: J65.4, J66.4, J67.4, J68.4
- new net SCL17: J69.4, J70.4, J71.4, J72.4
- new net SCL18: J73.4, J74.4, J75.4, J76.4
- new net SCL19: J77.4, J78.4, J79.4, J80.4
- new net SCL20: J81.4, J82.4, J83.4, J84.4
- new net SCL21: J85.4, J86.4, J87.4, J88.4
- new net SCL22: J89.4, J90.4, J91.4, J92.4
- new net SCL23: J93.4, J94.4, J95.4, J96.4
- new net SCL24: J100.4, J97.4, J98.4, J99.4
- new net SCL9: J37.4, J38.4, J39.4, J40.4
- new net SDA10: J41.3, J42.3, J43.3, J44.3
- new net SDA11: J45.3, J46.3, J47.3, J48.3
- new net SDA12: J49.3, J50.3, J51.3, J52.3
- new net SDA13: J53.3, J54.3, J55.3, J56.3
- new net SDA14: J57.3, J58.3, J59.3, J60.3
- new net SDA15: J61.3, J62.3, J63.3, J64.3
- new net SDA16: J65.3, J66.3, J67.3, J68.3
- new net SDA17: J69.3, J70.3, J71.3, J72.3
- new net SDA18: J73.3, J74.3, J75.3, J76.3
- new net SDA19: J77.3, J78.3, J79.3, J80.3
- new net SDA20: J81.3, J82.3, J83.3, J84.3
- new net SDA21: J85.3, J86.3, J87.3, J88.3
- new net SDA22: J89.3, J90.3, J91.3, J92.3
- new net SDA23: J93.3, J94.3, J95.3, J96.3
- new net SDA24: J100.3, J97.3, J98.3, J99.3
- new net SDA9: J37.3, J38.3, J39.3, J40.3
Routing:
- net SCL12: track 0.00 -> 43.5 mm, vias 0 -> 5
- net SCL10: track 0.00 -> 43.5 mm, vias 0 -> 5
- net SCL15: track 0.00 -> 43.5 mm, vias 0 -> 5
- net SCL11: track 0.00 -> 43.5 mm, vias 0 -> 5
- net SCL17: track 0.00 -> 43.5 mm, vias 0 -> 5
- net SCL16: track 0.00 -> 43.5 mm, vias 0 -> 5
- net SCL22: track 0.00 -> 43.5 mm, vias 0 -> 5
- net SCL20: track 0.00 -> 43.5 mm, vias 0 -> 5
- net SCL14: track 0.00 -> 43.5 mm, vias 0 -> 5
- net SCL13: track 0.00 -> 43.5 mm, vias 0 -> 5
- net SCL18: track 0.00 -> 43.5 mm, vias 0 -> 5
- net SCL21: track 0.00 -> 43.5 mm, vias 0 -> 5
- net SCL19: track 0.00 -> 43.5 mm, vias 0 -> 5
- net SCL9: track 0.00 -> 43.5 mm, vias 0 -> 5
- net SCL24: track 0.00 -> 43.5 mm, vias 0 -> 5
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- added copper zone on layer 1, net GND10
- added copper zone on layer 16, net GND10
- added copper zone on layer 1, net GND11
- added copper zone on layer 16, net GND11
- added copper zone on layer 1, net GND12
- added copper zone on layer 16, net GND12
- added copper zone on layer 1, net GND13
- added copper zone on layer 16, net GND13
- added copper zone on layer 1, net GND14
- added copper zone on layer 16, net GND14
- added copper zone on layer 1, net GND15
- added copper zone on layer 16, net GND15
- added copper zone on layer 1, net GND16
- added copper zone on layer 16, net GND16
- added copper zone on layer 1, net GND17
- added copper zone on layer 16, net GND17
- added copper zone on layer 1, net GND18
- added copper zone on layer 16, net GND18
- added copper zone on layer 1, net GND19
- added copper zone on layer 16, net GND19
- added copper zone on layer 1, net GND20
- added copper zone on layer 16, net GND20
- added copper zone on layer 1, net GND21
- added copper zone on layer 16, net GND21
- added copper zone on layer 1, net GND22
- added copper zone on layer 16, net GND22
- added copper zone on layer 1, net GND23
- added copper zone on layer 16, net GND23
- added copper zone on layer 1, net GND24
- added copper zone on layer 16, net GND24
- added copper zone on layer 1, net GND9
- added copper zone on layer 16, net GND9
Other:
- board size 97.3 x 97.3 mm -> 129 x 129 mm
- board text added: "Route out"
- board text removed: "v-score"
